File: pH.sch (KiCad schematic (older format))
At the start: 3 parts, among them U1 LMV341

Commit message: changed op amp from LMV341 to MCP6241
Parts:
- removed U1: LMV341, symbol LMV341
- added U1: MCP6241, ~, symbol MCP6241
Changed lines of the file:
@@
 Sheet 3 7
 Title ""
-Date "12 aug 2014"
+Date "14 aug 2014"
 Rev ""
 Comp ""
@@
 Text Label 4450 3100 0    60   ~ 0
 V+(in)
-$Comp
-L LMV341 U1
-U 1 1 53E268A2
-P 3800 3200
-F 0 "U1" H 3800 3350 60  0000 L CNN
-F 1 "LMV341" H 3800 3050 60  0000 L CNN
-F 2 "" H 3800 3200 60  0000 C CNN
-F 3 "" H 3800 3200 60  0000 C CNN
-	1    3800 3200
-	-1   0    0    -1
-$EndComp
 Text Label 3900 2750 0    60   ~ 0
 V+
@@
 pH_VGND
 Connection ~ 4450 3300
+$Comp
+L MCP6241 U1
+U 1 1 53ECAB65
+P 3800 3200
+F 0 "U1" H 3800 3350 60  0000 L CNN
+F 1 "MCP6241" H 3800 3050 60  0000 L CNN
+F 2 "~" H 3800 3200 60  0000 C CNN
+F 3 "~" H 3800 3200 60  0000 C CNN
+	1    3800 3200
+	-1   0    0    -1
+$EndComp
 $EndSCHEMATC
