File: Kicad/HealthyPH.kicad_pcb (KiCad board)
At the start: 2 copper layers, 68.6 x 53.4 mm, 35 parts, among them CON1 LB_BarrelJack, P1 CONN_8, P2 WallWartExtension, Q1 TIP122, Q2 TIP122, U1 MCP6241, U2 MCP3901, U3 MC78L05, X1 CRYSTAL

Commit message: Dev Rev 1
Parts:
- added D3: 4004, DO-214AC(SMA), F.Cu at (176.3, 101.8)
- added TP1: CONN_1, LB_TestPoint, F.Cu at (209.9, 83.6)
- added TP10: CONN_1, LB_TestPoint, F.Cu at (197.4, 91.8)
- added TP11: CONN_1, LB_TestPoint, F.Cu at (197.3, 85.9)
- added TP12: CONN_1, LB_TestPoint, F.Cu at (210.3, 91.4)
- added TP2: CONN_1, LB_TestPoint, F.Cu at (171.0, 71.6)
- added TP3: CONN_1, LB_TestPoint, F.Cu at (167.9, 71.7)
- added TP4: CONN_1, LB_TestPoint, F.Cu at (164.6, 71.7)
- added TP5: CONN_1, LB_TestPoint, F.Cu at (173.9, 71.7)
- added TP6: CONN_1, LB_TestPoint, F.Cu at (209.2, 74.7)
- added TP7: CONN_1, LB_TestPoint, F.Cu at (198.6, 71.7)
- added TP8: CONN_1, LB_TestPoint, F.Cu at (200.0, 90.2)
- added TP9: CONN_1, LB_TestPoint, F.Cu at (179.0, 108.1)
Connections:
- net /Pumps/PUMP renamed N-0000025
- C12 pad 1: N-0000034 (its old number) -> N-0000035
- C13 pad 1: N-0000034 (its old number) -> N-0000035
- P2 pad 2: /Digital Access/V+_WallWart -> N-0000035
- U3 pad 2: N-0000034 (its old number) -> N-0000035
Routing:
- net N-0000035: track 0.00 -> 29.1 mm
- net /Digital Access/MOSI_ISO: track 14.2 -> 38.5 mm, vias 0 -> 1
- net /Digital Access/~CS_ISO: track 13.6 -> 30.4 mm, vias 0 -> 1
- net N-0000034 (its old number): track 15.2 -> 0.00 mm
- net /Digital Access/MISO_ISO: track 18.1 -> 31.1 mm, vias 0 -> 1
- net /Digital Access/~DR: track 32.7 -> 43.4 mm
- net /Digital Access/SCLK_ISO: track 18.6 -> 26.3 mm
- net N-0000033: track 11.7 -> 17.0 mm
- net /Digital Access/V+_WallWart: track 77.2 -> 80.1 mm
- net /Arduino/~RESET: track 85.4 -> 88.1 mm
- net /Temperature/Temp: track 38.2 -> 40.7 mm
- net /Digital Access/pH_ADC-: track 34.1 -> 36.1 mm
- net /Digital Access/pH_ADC+: track 44.0 -> 46.0 mm
- net /Pumps/V+_DownPump: track 31.5 -> 33.2 mm

Commit message: updates for dev rev 2
Parts:
- moved CON1 0.55 mm to (149.0, 107.4)
Changed lines of the file:
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@@
     (links 90)
     (no_connects 0)
-    (area 150.931879 64.785239 219.656661 118.292881)
+    (area 144.330999 64.530999 219.919001 118.704)
     (thickness 1.6)
     (drawings 10)
@@
     (mod_text_size 1 1)
     (mod_text_width 0.15)
-    (pad_size 1.778 1.778)
-    (pad_drill 1.016)
+    (pad_size 1.5 1)
+    (pad_drill 1.1)
     (pad_to_mask_clearance 0)
     (aux_axis_origin 0 0)
@@
     )
   )
-  (module LB_BarrelJack (layer F.Cu)
-    (at 148.95 107.95)
-    (fp_text reference CON1 (at 6.5 -0.725) (layer F.SilkS)
-      (effects (font (size 1 1) (thickness 0.15)))
-    )
-    (fp_text value LB_BarrelJack (at 8.276 6.604) (layer F.SilkS)
-      (effects (font (size 1 1) (thickness 0.15)))
-    )
-    (fp_line (start 2 5.5) (end 2 5.7) (layer F.SilkS) (width 0.15))
-    (fp_line (start 2 0) (end 2 5.6) (layer F.SilkS) (width 0.15))
-    (fp_line (start 0.05 4.925) (end 0.05 5.75) (layer F.SilkS) (width 0.15))
-    (fp_line (start 0.05 5.75) (end 0.325 5.75) (layer F.SilkS) (width 0.15))
-    (fp_line (start 11.375 -0.05) (end 11.85 -0.05) (layer F.SilkS) (width 0.15))
-    (fp_line (start 11.85 4.9) (end 11.85 5.75) (layer F.SilkS) (width 0.15))
-    (fp_line (start 0.35 5.75) (end 11.75 5.75) (layer F.SilkS) (width 0.15))
-    (fp_line (start 11.85 4.95) (end 11.85 -0.05) (layer F.SilkS) (width 0.15))
-    (fp_line (start 11.45 -0.05) (end 0.05 -0.05) (layer F.SilkS) (width 0.15))
-    (fp_line (start 0.05 -0.05) (end 0.05 4.95) (layer F.SilkS) (width 0.15))
-    (pad 2 thru_hole oval (at 6.2 2.5 180) (size 0.3 1) (drill oval 0.3 1)
-      (layers *.Cu *.Mask F.SilkS)
-      (net 23 AGND)
-    )
-    (pad 3 thru_hole oval (at 8.7 5.2 180) (size 1 0.3) (drill oval 1 0.3)
-      (layers *.Cu *.Mask F.SilkS)
-      (net 23 AGND)
-    )
-    (pad 1 thru_hole oval (at 11.2 2.5 180) (size 0.3 1) (drill oval 0.3 1)
-      (layers *.Cu *.Mask F.SilkS)
-      (net 32 N-0000034)
-    )
-  )
   (module "DO-214AC(SMA)" (layer F.Cu)
     (at 191.05 98.85)
@@
       (layers *.Cu *.Mask F.SilkS)
       (net 14 "/Digital Access/pH_ADC-")
+    )
+  )
+  (module LB_BarrelJack (layer F.Cu)
+    (at 149 107.4)
+    (fp_text reference CON1 (at 6.5 -0.725) (layer F.SilkS)
+      (effects (font (size 1 1) (thickness 0.15)))
+    )
+    (fp_text value LB_BarrelJack (at 8.276 6.604) (layer F.SilkS)
+      (effects (font (size 1 1) (thickness 0.15)))
+    )
+    (fp_line (start 2 5.5) (end 2 5.7) (layer F.SilkS) (width 0.15))
+    (fp_line (start 2 0) (end 2 5.6) (layer F.SilkS) (width 0.15))
+    (fp_line (start 0.05 4.925) (end 0.05 5.75) (layer F.SilkS) (width 0.15))
+    (fp_line (start 0.05 5.75) (end 0.325 5.75) (layer F.SilkS) (width 0.15))
+    (fp_line (start 11.375 -0.05) (end 11.85 -0.05) (layer F.SilkS) (width 0.15))
+    (fp_line (start 11.85 4.9) (end 11.85 5.75) (layer F.SilkS) (width 0.15))
+    (fp_line (start 0.35 5.75) (end 11.75 5.75) (layer F.SilkS) (width 0.15))
+    (fp_line (start 11.85 4.95) (end 11.85 -0.05) (layer F.SilkS) (width 0.15))
+    (fp_line (start 11.45 -0.05) (end 0.05 -0.05) (layer F.SilkS) (width 0.15))
+    (fp_line (start 0.05 -0.05) (end 0.05 4.95) (layer F.SilkS) (width 0.15))
+    (pad 2 thru_hole oval (at 6.2 2.7 180) (size 1 1.5) (drill oval 0.4 1.1)
+      (layers *.Cu *.Mask F.SilkS)
+      (net 23 AGND)
+    )
+    (pad 3 thru_hole oval (at 8.7 4.9 180) (size 1.5 1) (drill oval 1.1 0.4)
+      (layers *.Cu *.Mask F.SilkS)
+      (net 23 AGND)
+    )
+    (pad 1 thru_hole oval (at 10.9 2.8 180) (size 1 1.5) (drill oval 0.4 1.1)
+      (layers *.Cu *.Mask F.SilkS)
+      (net 32 N-0000034)
     )
   )
@@
   (segment (start 184.02 96.5575) (end 180.5285 96.5575) (width 0.254) (layer F.Cu) (net 30) (status 30))
   (segment (start 180.5285 96.5575) (end 179.93 95.959) (width 0.254) (layer F.Cu) (net 30) (status 30))
-  (segment (start 178.9938 108.1278) (end 173.9378 108.1278) (width 0.254) (layer F.Cu) (net 31) (status 400000))
+  (segment (start 178.9938 108.1278) (end 173.9378 108.1278) (width 0.254) (layer F.Cu) (net 31))
   (segment (start 173.9378 108.1278) (end 173.75114 107.94114) (width 0.254) (layer F.Cu) (net 31))
   (segment (start 173.75114 105.27666) (end 173.75114 107.94114) (width 0.254) (layer F.Cu) (net 31) (status 10))
@@
   (zone (net 23) (net_name AGND) (layer B.Cu) (hatch edge 0.508)
     (connect_pads (clearance 0.508))
-    (min_thickness 0.254)
-    (fill (arc_segments 16) (thermal_gap 0.508) (thermal_bridge_width 0.508))
+    (min_thickness 0.0254)
+    (fill (arc_segments 16) (thermal_gap 1.016) (thermal_bridge_width 0.2286))
     (polygon
       (pts
