File: Kicad/Arduino.sch (KiCad schematic (older format))
At the start: 1 part

Commit message: updates for dev rev 2
Parts:
- added D?: LED, ~, symbol LED
- added R?: 125, ~, symbol R
Connections:
- net GND_ARD: now also D?.2 (K)
- net at ARD1.14 (Digital3): now also R?.1
- net TempV: now reaches ARD1.7 (AnalogIn2)
- new net: D?.1 (A), R?.2
Changed lines of the file:
@@
 Sheet 5 7
 Title ""
-Date "21 aug 2014"
+Date "9 sep 2014"
 Rev ""
 Comp ""
@@
 Wire Wire Line
 	5750 3800 6400 3800
+Text HLabel 2500 3950 0    60   Input ~ 0
+TempV
+Wire Wire Line
+	3550 3950 2500 3950
+$Comp
+L R R?
+U 1 1 540EE433
+P 6400 4000
+F 0 "R?" V 6480 4000 40  0000 C CNN
+F 1 "125" V 6407 4001 40  0000 C CNN
+F 2 "~" V 6330 4000 30  0000 C CNN
+F 3 "~" H 6400 4000 30  0000 C CNN
+	1    6400 4000
+	0    -1   -1   0
+$EndComp
+Wire Wire Line
+	5750 4000 6150 4000
+Wire Wire Line
+	6650 4000 6850 4000
+Wire Wire Line
+	6850 4900 3100 4900
+Wire Wire Line
+	3100 4900 3100 2650
+Connection ~ 3100 2650
+$Comp
+L LED D?
+U 1 1 540EE47C
+P 6850 4400
+F 0 "D?" H 6850 4500 50  0000 C CNN
+F 1 "LED" H 6850 4300 50  0000 C CNN
+F 2 "~" H 6850 4400 60  0000 C CNN
+F 3 "~" H 6850 4400 60  0000 C CNN
+	1    6850 4400
+	0    1    1    0
+$EndComp
+Wire Wire Line
+	6850 4000 6850 4200
+Wire Wire Line
+	6850 4600 6850 4900
+Text Label 7050 4350 0    60   ~ 0
+RGB Circuit Status
+Text Label 7050 4500 0    60   ~ 0
+I=20mA, Vf = 2.5V
+Text Label 5850 3950 0    60   ~ 0
+5V
+Text Label 6700 3950 0    60   ~ 0
+2.5V
 $EndSCHEMATC

Commit message: Ready for Schematic Design Review
Parts:
- removed D?: LED, ~, symbol LED
- removed R?: 125, ~, symbol R
- added D4: RGB_LED, ~, symbol RGB_LED
- added R12, R13, R14: 500, ~, symbol R
Connections:
- net V+_ARD: now also D4.4
- net ~CS: now also ARD1.19 (Digital8); no longer ARD1.21 (CS_N)
- net at ARD1.17 (Digital6): now also R14.1
- net at ARD1.20 (PWM0): now also R13.1
- net TempV: no longer names the net of ARD1.7 (AnalogIn2)
- new net: ARD1.21 (CS_N), R12.1
- new net: D4.1 (A1), R12.2
- new net: D4.2, R13.2
- new net: D4.3, R14.2
Changed lines of the file:
@@
 $Descr A4 11693 8268
 encoding utf-8
-Sheet 5 7
+Sheet 3 7
 Title ""
-Date "9 sep 2014"
+Date "10 sep 2014"
 Rev ""
 Comp ""
@@
 Text HLabel 6350 2400 2    60   Output ~ 0
 MOSI
-Text HLabel 6350 2600 2    60   Output ~ 0
+Text HLabel 6350 3000 2    60   Output ~ 0
 ~CS
 Wire Wire Line
@@
 	5750 2400 6350 2400
 Wire Wire Line
-	5750 2600 6350 2600
+	5750 3000 6350 3000
 Text HLabel 2500 3550 0    60   Output ~ 0
 PumpDown
@@
 Wire Wire Line
 	5750 3800 6400 3800
-Text HLabel 2500 3950 0    60   Input ~ 0
-TempV
+$Comp
+L RGB_LED D4
+U 1 1 540F4D9B
+P 7700 3100
+F 0 "D4" H 7800 3450 50  0000 L CNN
+F 1 "RGB_LED" H 7700 2500 50  0000 C CNN
+F 2 "~" H 7700 3100 60  0000 C CNN
+F 3 "~" H 7700 3100 60  0000 C CNN
+	1    7700 3100
+	-1   0    0    1
+$EndComp
 Wire Wire Line
-	3550 3950 2500 3950
+	3150 2450 3150 900
+Wire Wire Line
+	3150 900  8100 900
+Wire Wire Line
+	8100 900  8100 3000
+Connection ~ 3150 2450
+Wire Wire Line
+	7350 2800 7350 2600
+Wire Wire Line
+	7350 3000 7200 3000
+Wire Wire Line
+	7200 3000 7200 2800
+Wire Wire Line
+	7350 3400 7350 3200
 $Comp
-L R R?
-U 1 1 540EE433
-P 6400 4000
-F 0 "R?" V 6480 4000 40  0000 C CNN
-F 1 "125" V 6407 4001 40  0000 C CNN
-F 2 "~" V 6330 4000 30  0000 C CNN
-F 3 "~" H 6400 4000 30  0000 C CNN
-	1    6400 4000
+L R R14
+U 1 1 540F4E5D
+P 6500 3400
+F 0 "R14" V 6580 3400 40  0000 C CNN
+F 1 "500" V 6507 3401 40  0000 C CNN
+F 2 "~" V 6430 3400 30  0000 C CNN
+F 3 "~" H 6500 3400 30  0000 C CNN
+	1    6500 3400
 	0    -1   -1   0
 $EndComp
 Wire Wire Line
-	5750 4000 6150 4000
+	5750 3400 6250 3400
 Wire Wire Line
-	6650 4000 6850 4000
-Wire Wire Line
-	6850 4900 3100 4900
-Wire Wire Line
-	3100 4900 3100 2650
-Connection ~ 3100 2650
+	6750 3400 7350 3400
 $Comp
-L LED D?
-U 1 1 540EE47C
-P 6850 4400
-F 0 "D?" H 6850 4500 50  0000 C CNN
-F 1 "LED" H 6850 4300 50  0000 C CNN
-F 2 "~" H 6850 4400 60  0000 C CNN
-F 3 "~" H 6850 4400 60  0000 C CNN
-	1    6850 4400
-	0    1    1    0
+L R R13
+U 1 1 540F4E9E
+P 6500 2800
+F 0 "R13" V 6580 2800 40  0000 C CNN
+F 1 "500" V 6507 2801 40  0000 C CNN
+F 2 "~" V 6430 2800 30  0000 C CNN
+F 3 "~" H 6500 2800 30  0000 C CNN
+	1    6500 2800
+	0    -1   -1   0
 $EndComp
 Wire Wire Line
-	6850 4000 6850 4200
+	5750 2800 6250 2800
 Wire Wire Line
-	6850 4600 6850 4900
-Text Label 7050 4350 0    60   ~ 0
-RGB Circuit Status
-Text Label 7050 4500 0    60   ~ 0
-I=20mA, Vf = 2.5V
-Text Label 5850 3950 0    60   ~ 0
-5V
-Text Label 6700 3950 0    60   ~ 0
-2.5V
+	7200 2800 6750 2800
+$Comp
+L R R12
+U 1 1 540F4F03
+P 6500 2600
+F 0 "R12" V 6580 2600 40  0000 C CNN
+F 1 "500" V 6507 2601 40  0000 C CNN
+F 2 "~" V 6430 2600 30  0000 C CNN
+F 3 "~" H 6500 2600 30  0000 C CNN
+	1    6500 2600
+	0    -1   -1   0
+$EndComp
+Wire Wire Line
+	6250 2600 5750 2600
+Wire Wire Line
+	7350 2600 6750 2600
 $EndSCHEMATC

Commit message: updated 500R to 499R
Parts:
- R12, R13, R14: value 500 -> 499
Changed lines of the file:
@@
 Sheet 3 7
 Title ""
-Date "10 sep 2014"
+Date "11 sep 2014"
 Rev ""
 Comp ""
@@
 P 6500 3400
 F 0 "R14" V 6580 3400 40  0000 C CNN
-F 1 "500" V 6507 3401 40  0000 C CNN
+F 1 "499" V 6507 3401 40  0000 C CNN
 F 2 "~" V 6430 3400 30  0000 C CNN
 F 3 "~" H 6500 3400 30  0000 C CNN
@@
 P 6500 2800
 F 0 "R13" V 6580 2800 40  0000 C CNN
-F 1 "500" V 6507 2801 40  0000 C CNN
+F 1 "499" V 6507 2801 40  0000 C CNN
 F 2 "~" V 6430 2800 30  0000 C CNN
 F 3 "~" H 6500 2800 30  0000 C CNN
@@
 P 6500 2600
 F 0 "R12" V 6580 2600 40  0000 C CNN
-F 1 "500" V 6507 2601 40  0000 C CNN
+F 1 "499" V 6507 2601 40  0000 C CNN
 F 2 "~" V 6430 2600 30  0000 C CNN
 F 3 "~" H 6500 2600 30  0000 C CNN

Commit message: layout sent to OshPark
Connections:
- net ~CS: now also ARD1.21 (CS_N); no longer ARD1.19 (Digital8)
- net at ARD1.17 (Digital6): no longer R14.1
- net at ARD1.20 (PWM0): no longer R13.1
- net at R12.1: now also D4.1 (A1); no longer ARD1.21 (CS_N)
- net at ARD1.7 (AnalogIn2): now also R12.2
- net at ARD1.8 (AnalogIn3): now also R13.2
- net at ARD1.9 (SDA): now also R14.2
- net at D4.2: now also R14.1; no longer R13.2
- net at D4.3: now also R13.1; no longer R14.2
Other:
- moved on the sheet: D4, R12, R13, R14
Changed lines of the file:
@@
 Sheet 3 7
 Title ""
-Date "13 sep 2014"
+Date "15 sep 2014"
 Rev ""
 Comp ""
@@
 Text HLabel 6350 2400 2    60   Output ~ 0
 MOSI
-Text HLabel 6350 3000 2    60   Output ~ 0
+Text HLabel 6350 2600 2    60   Output ~ 0
 ~CS
 Wire Wire Line
@@
 Wire Wire Line
 	5750 2400 6350 2400
-Wire Wire Line
-	5750 3000 6350 3000
 Text HLabel 2500 3550 0    60   Output ~ 0
 PumpDown
@@
 L RGB_LED D4
 U 1 1 540F4D9B
-P 7700 3100
-F 0 "D4" H 7800 3450 50  0000 L CNN
-F 1 "RGB_LED" H 7700 2500 50  0000 C CNN
-F 2 "~" H 7700 3100 60  0000 C CNN
-F 3 "~" H 7700 3100 60  0000 C CNN
-	1    7700 3100
-	-1   0    0    1
+P 1750 4250
+F 0 "D4" H 1850 4600 50  0000 L CNN
+F 1 "RGB_LED" H 1750 3650 50  0000 C CNN
+F 2 "~" H 1750 4250 60  0000 C CNN
+F 3 "~" H 1750 4250 60  0000 C CNN
+	1    1750 4250
+	1    0    0    1
 $EndComp
-Wire Wire Line
-	3150 2450 3150 900
-Wire Wire Line
-	3150 900  8100 900
-Wire Wire Line
-	8100 900  8100 3000
-Connection ~ 3150 2450
-Wire Wire Line
-	7350 2800 7350 2600
-Wire Wire Line
-	7350 3000 7200 3000
-Wire Wire Line
-	7200 3000 7200 2800
-Wire Wire Line
-	7350 3400 7350 3200
 $Comp
 L R R14
 U 1 1 540F4E5D
-P 6500 3400
-F 0 "R14" V 6580 3400 40  0000 C CNN
-F 1 "499" V 6507 3401 40  0000 C CNN
-F 2 "~" V 6430 3400 30  0000 C CNN
-F 3 "~" H 6500 3400 30  0000 C CNN
-	1    6500 3400
+P 2850 4150
+F 0 "R14" V 2930 4150 40  0000 C CNN
+F 1 "499" V 2857 4151 40  0000 C CNN
+F 2 "~" V 2780 4150 30  0000 C CNN
+F 3 "~" H 2850 4150 30  0000 C CNN
+	1    2850 4150
+	0    -1   -1   0
+$EndComp
+$Comp
+L R R13
+U 1 1 540F4E9E
+P 2850 4350
+F 0 "R13" V 2930 4350 40  0000 C CNN
+F 1 "499" V 2857 4351 40  0000 C CNN
+F 2 "~" V 2780 4350 30  0000 C CNN
+F 3 "~" H 2850 4350 30  0000 C CNN
+	1    2850 4350
+	0    -1   -1   0
+$EndComp
+$Comp
+L R R12
+U 1 1 540F4F03
+P 2850 3950
+F 0 "R12" V 2930 3950 40  0000 C CNN
+F 1 "499" V 2857 3951 40  0000 C CNN
+F 2 "~" V 2780 3950 30  0000 C CNN
+F 3 "~" H 2850 3950 30  0000 C CNN
+	1    2850 3950
 	0    -1   -1   0
 $EndComp
 Wire Wire Line
-	5750 3400 6250 3400
+	5750 2600 6350 2600
 Wire Wire Line
-	6750 3400 7350 3400
-$Comp
-L R R13
-U 1 1 540F4E9E
-P 6500 2800
-F 0 "R13" V 6580 2800 40  0000 C CNN
-F 1 "499" V 6507 2801 40  0000 C CNN
-F 2 "~" V 6430 2800 30  0000 C CNN
-F 3 "~" H 6500 2800 30  0000 C CNN
-	1    6500 2800
-	0    -1   -1   0
-$EndComp
+	3550 3950 3100 3950
 Wire Wire Line
-	5750 2800 6250 2800
+	2600 3950 2100 3950
 Wire Wire Line
-	7200 2800 6750 2800
-$Comp
-L R R12
-U 1 1 540F4F03
-P 6500 2600
-F 0 "R12" V 6580 2600 40  0000 C CNN
-F 1 "499" V 6507 2601 40  0000 C CNN
-F 2 "~" V 6430 2600 30  0000 C CNN
-F 3 "~" H 6500 2600 30  0000 C CNN
-	1    6500 2600
-	0    -1   -1   0
-$EndComp
+	2600 4150 2100 4150
 Wire Wire Line
-	6250 2600 5750 2600
+	2600 4350 2100 4350
 Wire Wire Line
-	7350 2600 6750 2600
+	1350 4150 1200 4150
+Text HLabel 1200 4150 0    60   Output ~ 0
+V+_ARD
+Wire Wire Line
+	3100 4150 3200 4150
+Wire Wire Line
+	3200 4150 3200 4350
+Wire Wire Line
+	3200 4350 3550 4350
+Wire Wire Line
+	3100 4350 3100 4250
+Wire Wire Line
+	3100 4250 3550 4250
+Wire Wire Line
+	3550 4250 3550 4150
 $EndSCHEMATC
