File: Kicad/Pumps.sch (KiCad schematic (older format))
At the start: 6 parts, among them Q1 TIP122, Q2 TIP122

Commit message: Layout with traces - ran through ERC and DRC
Connections:
- net PUMP: no longer Q2.1 (B), R11.2
- net V+_ARD: now also D1.1 (A); no longer D1.2 (K)
- net V+_DownPump: now also D1.2 (K); no longer D1.1 (A)
- new net: Q2.1 (B), R11.2
Changed lines of the file:
@@
 Sheet 7 7
 Title ""
-Date "14 aug 2014"
+Date "19 aug 2014"
 Rev ""
 Comp ""
@@
 F 3 "~" H 4700 1500 60  0000 C CNN
 	1    4700 1500
-	0    -1   -1   0
+	0    1    1    0
 $EndComp
 Wire Wire Line
@@
 DownPump
 $Comp
-L GND #PWR13
+L GND #PWR013
 U 1 1 53DC3138
 P 3900 3250
-F 0 "#PWR13" H 3900 3250 30  0001 C CNN
+F 0 "#PWR013" H 3900 3250 30  0001 C CNN
 F 1 "GND" H 3900 3180 30  0001 C CNN
 F 2 "" H 3900 3250 60  0000 C CNN
@@
 Wire Wire Line
 	1750 1150 4700 1150
-Text Label 4050 2350 0    60   ~ 0
-SW-DownPump
 Text Label 4700 1900 0    60   ~ 0
 Pump-V+
@@
 Connection ~ 2800 1150
 $Comp
-L GND #PWR12
+L GND #PWR014
 U 1 1 53E3E3F6
 P 2800 1850
-F 0 "#PWR12" H 2800 1850 30  0001 C CNN
+F 0 "#PWR014" H 2800 1850 30  0001 C CNN
 F 1 "GND" H 2800 1780 30  0001 C CNN
 F 2 "" H 2800 1850 60  0000 C CNN
@@
 Wire Wire Line
 	2800 1700 2800 1850
-Text Label 3900 3000 0    60   ~ 0
-Pump-GND
 Text HLabel 6000 2150 2    60   Input ~ 0
 V+_DownPump
@@
 UpPump
 $Comp
-L GND #PWR14
+L GND #PWR015
 U 1 1 53EA6E1E
 P 3900 4750
-F 0 "#PWR14" H 3900 4750 30  0001 C CNN
+F 0 "#PWR015" H 3900 4750 30  0001 C CNN
 F 1 "GND" H 3900 4680 30  0001 C CNN
 F 2 "" H 3900 4750 60  0000 C CNN
@@
 Wire Wire Line
 	3900 3850 3900 3950
-Text Label 4050 3850 0    60   ~ 0
-SW_UpPump
-Text Label 3450 4150 0    60   ~ 0
-PUMP
 Wire Wire Line
 	3900 4350 3900 4750
-Text Label 3900 4500 0    60   ~ 0
-Pump-GND
 Text HLabel 6000 3850 2    60   Input ~ 0
 SW_UpPump

Commit message: Dev Rev 1
Connections:
- net PUMP: no longer names the net of Q1.1 (B), R1.2
Changed lines of the file:
@@
 Sheet 7 7
 Title ""
-Date "20 aug 2014"
+Date "21 aug 2014"
 Rev ""
 Comp ""
@@
 Wire Wire Line
 	1750 1150 4700 1150
-Text Label 4700 1900 0    60   ~ 0
-Pump-V+
-Text Label 3450 2650 0    60   ~ 0
-PUMP
 Wire Wire Line
 	3900 2850 3900 3250

Commit message: updates for dev rev 2
Parts:
- removed C14: 1u, ~, symbol C
- added D?: 4004, ~, symbol DIODE
Connections:
- net V+_DownPump is gone; now on net V+_ARD: D1.2 (K)
- net SW_DownPump: now also D1.1 (A)
- net SW_UpPump: now also D?.1 (A)
- net V+_ARD: now also D?.2 (K); no longer D1.1 (A)
Other:
- moved on the sheet: D1
Changed lines of the file:
@@
 Sheet 7 7
 Title ""
-Date "21 aug 2014"
+Date "9 sep 2014"
 Rev ""
 Comp ""
@@
 L DIODE D1
 U 1 1 53CBD4B8
-P 4700 1500
-F 0 "D1" H 4700 1600 40  0000 C CNN
-F 1 "4004" H 4700 1400 40  0000 C CNN
-F 2 "~" H 4700 1500 60  0000 C CNN
-F 3 "~" H 4700 1500 60  0000 C CNN
-	1    4700 1500
-	0    1    1    0
+P 5650 2050
+F 0 "D1" H 5650 2150 40  0000 C CNN
+F 1 "4004" H 5650 1950 40  0000 C CNN
+F 2 "~" H 5650 2050 60  0000 C CNN
+F 3 "~" H 5650 2050 60  0000 C CNN
+	1    5650 2050
+	0    -1   -1   0
 $EndComp
-Wire Wire Line
-	4700 1150 4700 1300
 Text HLabel 2000 2650 0    59   Input ~ 0
 DownPump
@@
 	1    0    0    -1
 $EndComp
-Text HLabel 1750 1150 0    60   Input ~ 0
+Text HLabel 1750 1700 0    60   Input ~ 0
 V+_ARD
 Wire Wire Line
@@
 	3900 2350 3900 2450
 Wire Wire Line
-	4700 1700 4700 2150
-Wire Wire Line
-	4700 2150 6000 2150
-$Comp
-L C C14
-U 1 1 53E26DDA
-P 2800 1500
-F 0 "C14" H 2800 1600 40  0000 L CNN
-F 1 "1u" H 2806 1415 40  0000 L CNN
-F 2 "~" H 2838 1350 30  0000 C CNN
-F 3 "~" H 2800 1500 60  0000 C CNN
-	1    2800 1500
-	-1   0    0    1
-$EndComp
-Wire Wire Line
-	1750 1150 4700 1150
+	1750 1700 6000 1700
 Wire Wire Line
 	3900 2850 3900 3250
@@
 	2000 3150 3900 3150
 Connection ~ 3900 3150
-Wire Wire Line
-	2800 1300 2800 1150
-Connection ~ 2800 1150
-$Comp
-L GND #PWR014
-U 1 1 53E3E3F6
-P 2800 1850
-F 0 "#PWR014" H 2800 1850 30  0001 C CNN
-F 1 "GND" H 2800 1780 30  0001 C CNN
-F 2 "" H 2800 1850 60  0000 C CNN
-F 3 "" H 2800 1850 60  0000 C CNN
-	1    2800 1850
-	1    0    0    -1
-$EndComp
-Wire Wire Line
-	2800 1700 2800 1850
-Text HLabel 6000 2150 2    60   Input ~ 0
+Text HLabel 6000 1700 2    60   Input ~ 0
 V+_DownPump
 Text HLabel 6000 2350 2    60   Input ~ 0
@@
 SW_UpPump
 Wire Wire Line
-	5300 2150 5300 3500
+	5300 1700 5300 3200
 Wire Wire Line
-	5300 3500 6000 3500
-Connection ~ 5300 2150
-Text HLabel 6000 3500 2    60   Input ~ 0
+	5300 3200 6000 3200
+Connection ~ 5300 1700
+Text HLabel 6000 3200 2    60   Input ~ 0
 V+_UpPump
 Wire Wire Line
@@
 Connection ~ 3900 4600
 Connection ~ 2550 3150
+Text Label 2600 2400 0    60   ~ 0
+HIGH Signal -->
+Text Label 4150 3100 1    60   ~ 0
+<--
+Text Label 4150 2800 1    60   ~ 0
+Current
+$Comp
+L DIODE D?
+U 1 1 540E4757
+P 5650 3550
+F 0 "D?" H 5650 3650 40  0000 C CNN
+F 1 "4004" H 5650 3450 40  0000 C CNN
+F 2 "~" H 5650 3550 60  0000 C CNN
+F 3 "~" H 5650 3550 60  0000 C CNN
+	1    5650 3550
+	0    -1   -1   0
+$EndComp
+Wire Wire Line
+	5650 3350 5650 3200
+Connection ~ 5650 3200
+Wire Wire Line
+	5650 3750 5650 3850
+Connection ~ 5650 3850
+Wire Wire Line
+	5650 1850 5650 1700
+Connection ~ 5650 1700
+Wire Wire Line
+	5650 2250 5650 2350
+Connection ~ 5650 2350
+Text Label 5950 2100 0    60   ~ 0
+Stop Reverse Voltage Spike When Switched Off
 $EndSCHEMATC

Commit message: Ready for Schematic Design Review
Parts:
- added TP12, TP13, TP14, TP15, TP16: CONN_1, symbol CONN_1
- gave numbers to parts that had none: 1
Connections:
- net SW_DownPump: now also TP15.1
- net SW_UpPump: now also TP16.1
- net V+_ARD: now also TP14.1
- net at Q1.1 (B), R1.2: now also TP12.1
- net at Q2.1 (B), R11.2: now also TP13.1
Changed lines of the file:
@@
 $Descr A4 11693 8268
 encoding utf-8
-Sheet 7 7
+Sheet 5 7
 Title ""
-Date "9 sep 2014"
+Date "10 sep 2014"
 Rev ""
 Comp ""
@@
 	0    -1   -1   0
 $EndComp
-Wire Wire Line
-	3350 2650 3600 2650
-Wire Wire Line
-	2000 2650 2850 2650
 $Comp
 L DIODE D1
@@
 DownPump
 $Comp
-L GND #PWR013
+L GND #PWR05
 U 1 1 53DC3138
 P 3900 3250
-F 0 "#PWR013" H 3900 3250 30  0001 C CNN
+F 0 "#PWR05" H 3900 3250 30  0001 C CNN
 F 1 "GND" H 3900 3180 30  0001 C CNN
 F 2 "" H 3900 3250 60  0000 C CNN
@@
 Text HLabel 1750 1700 0    60   Input ~ 0
 V+_ARD
-Wire Wire Line
-	3900 2350 6000 2350
-Wire Wire Line
-	3900 2350 3900 2450
-Wire Wire Line
-	1750 1700 6000 1700
-Wire Wire Line
-	3900 2850 3900 3250
 Text HLabel 2000 3150 0    59   Output ~ 0
 GND_ARD
-Wire Wire Line
-	2000 3150 3900 3150
-Connection ~ 3900 3150
 Text HLabel 6000 1700 2    60   Input ~ 0
 V+_DownPump
@@
 	0    -1   -1   0
 $EndComp
-Wire Wire Line
-	3350 4150 3600 4150
-Wire Wire Line
-	2000 4150 2850 4150
 Text HLabel 2000 4150 0    59   Input ~ 0
 UpPump
 $Comp
-L GND #PWR015
+L GND #PWR06
 U 1 1 53EA6E1E
 P 3900 4750
-F 0 "#PWR015" H 3900 4750 30  0001 C CNN
+F 0 "#PWR06" H 3900 4750 30  0001 C CNN
 F 1 "GND" H 3900 4680 30  0001 C CNN
 F 2 "" H 3900 4750 60  0000 C CNN
@@
 	1    0    0    -1
 $EndComp
-Wire Wire Line
-	3900 3850 6000 3850
-Wire Wire Line
-	3900 3850 3900 3950
-Wire Wire Line
-	3900 4350 3900 4750
 Text HLabel 6000 3850 2    60   Input ~ 0
 SW_UpPump
-Wire Wire Line
-	5300 1700 5300 3200
-Wire Wire Line
-	5300 3200 6000 3200
-Connection ~ 5300 1700
 Text HLabel 6000 3200 2    60   Input ~ 0
 V+_UpPump
-Wire Wire Line
-	2550 3150 2550 4600
-Wire Wire Line
-	2550 4600 3900 4600
-Connection ~ 3900 4600
-Connection ~ 2550 3150
-Text Label 2600 2400 0    60   ~ 0
-HIGH Signal -->
-Text Label 4150 3100 1    60   ~ 0
-<--
-Text Label 4150 2800 1    60   ~ 0
-Current
-$Comp
-L DIODE D?
+$Comp
+L DIODE D5
 U 1 1 540E4757
 P 5650 3550
-F 0 "D?" H 5650 3650 40  0000 C CNN
+F 0 "D5" H 5650 3650 40  0000 C CNN
 F 1 "4004" H 5650 3450 40  0000 C CNN
 F 2 "~" H 5650 3550 60  0000 C CNN
@@
 	0    -1   -1   0
 $EndComp
+$Comp
+L CONN_1 TP14
+U 1 1 541050CF
+P 3750 1300
+F 0 "TP14" H 3830 1300 40  0000 L CNN
+F 1 "CONN_1" H 3750 1355 30  0001 C CNN
+F 2 "" H 3750 1300 60  0000 C CNN
+F 3 "" H 3750 1300 60  0000 C CNN
+	1    3750 1300
+	1    0    0    -1
+$EndComp
+$Comp
+L CONN_1 TP15
+U 1 1 54105105
+P 4650 2100
+F 0 "TP15" H 4730 2100 40  0000 L CNN
+F 1 "CONN_1" H 4650 2155 30  0001 C CNN
+F 2 "" H 4650 2100 60  0000 C CNN
+F 3 "" H 4650 2100 60  0000 C CNN
+	1    4650 2100
+	1    0    0    -1
+$EndComp
+$Comp
+L CONN_1 TP16
+U 1 1 5410510B
+P 4750 3500
+F 0 "TP16" H 4830 3500 40  0000 L CNN
+F 1 "CONN_1" H 4750 3555 30  0001 C CNN
+F 2 "" H 4750 3500 60  0000 C CNN
+F 3 "" H 4750 3500 60  0000 C CNN
+	1    4750 3500
+	1    0    0    -1
+$EndComp
+$Comp
+L CONN_1 TP13
+U 1 1 54105111
+P 3650 3650
+F 0 "TP13" H 3730 3650 40  0000 L CNN
+F 1 "CONN_1" H 3650 3705 30  0001 C CNN
+F 2 "" H 3650 3650 60  0000 C CNN
+F 3 "" H 3650 3650 60  0000 C CNN
+	1    3650 3650
+	1    0    0    -1
+$EndComp
+$Comp
+L CONN_1 TP12
+U 1 1 54105117
+P 3650 2100
+F 0 "TP12" H 3730 2100 40  0000 L CNN
+F 1 "CONN_1" H 3650 2155 30  0001 C CNN
+F 2 "" H 3650 2100 60  0000 C CNN
+F 3 "" H 3650 2100 60  0000 C CNN
+	1    3650 2100
+	1    0    0    -1
+$EndComp
+Wire Wire Line
+	3350 2650 3600 2650
+Wire Wire Line
+	2000 2650 2850 2650
+Wire Wire Line
+	3900 2350 6000 2350
+Wire Wire Line
+	3900 2350 3900 2450
+Wire Wire Line
+	1750 1700 6000 1700
+Wire Wire Line
+	3900 2850 3900 3250
+Wire Wire Line
+	2000 3150 3900 3150
+Connection ~ 3900 3150
+Wire Wire Line
+	3350 4150 3600 4150
+Wire Wire Line
+	2000 4150 2850 4150
+Wire Wire Line
+	3900 3850 6000 3850
+Wire Wire Line
+	3900 3850 3900 3950
+Wire Wire Line
+	3900 4350 3900 4750
+Wire Wire Line
+	5300 1700 5300 3200
+Wire Wire Line
+	5300 3200 6000 3200
+Connection ~ 5300 1700
+Wire Wire Line
+	2550 3150 2550 4600
+Wire Wire Line
+	2550 4600 3900 4600
+Connection ~ 3900 4600
+Connection ~ 2550 3150
 Wire Wire Line
 	5650 3350 5650 3200
@@
 	5650 2250 5650 2350
 Connection ~ 5650 2350
-Text Label 5950 2100 0    60   ~ 0
-Stop Reverse Voltage Spike When Switched Off
+Wire Wire Line
+	3600 1300 3600 1700
+Connection ~ 3600 1700
+Wire Wire Line
+	4500 2100 4500 2350
+Connection ~ 4500 2350
+Wire Wire Line
+	4600 3500 4600 3850
+Connection ~ 4600 3850
+Wire Wire Line
+	3500 2100 3500 2650
+Connection ~ 3500 2650
+Wire Wire Line
+	3500 3650 3500 4150
+Connection ~ 3500 4150
 $EndSCHEMATC
