File: Kicad/Pumps.sch (KiCad schematic (older format))
At the start: 11 parts, among them Q1 TIP122, Q2 TIP122

Commit message: Ready for Rev3 First layout review
Parts:
- removed TP12, TP13, TP14, TP15, TP16: CONN_1, symbol CONN_1
Changed lines of the file:
@@
 Sheet 5 7
 Title ""
-Date "11 oct 2014"
+Date "18 oct 2014"
 Rev ""
 Comp ""
@@
 	0    -1   -1   0
 $EndComp
-$Comp
-L CONN_1 TP14
-U 1 1 541050CF
-P 3750 1300
-F 0 "TP14" H 3830 1300 40  0000 L CNN
-F 1 "CONN_1" H 3750 1355 30  0001 C CNN
-F 2 "" H 3750 1300 60  0000 C CNN
-F 3 "" H 3750 1300 60  0000 C CNN
-	1    3750 1300
-	1    0    0    -1
-$EndComp
-$Comp
-L CONN_1 TP15
-U 1 1 54105105
-P 4650 2100
-F 0 "TP15" H 4730 2100 40  0000 L CNN
-F 1 "CONN_1" H 4650 2155 30  0001 C CNN
-F 2 "" H 4650 2100 60  0000 C CNN
-F 3 "" H 4650 2100 60  0000 C CNN
-	1    4650 2100
-	1    0    0    -1
-$EndComp
-$Comp
-L CONN_1 TP16
-U 1 1 5410510B
-P 4750 3500
-F 0 "TP16" H 4830 3500 40  0000 L CNN
-F 1 "CONN_1" H 4750 3555 30  0001 C CNN
-F 2 "" H 4750 3500 60  0000 C CNN
-F 3 "" H 4750 3500 60  0000 C CNN
-	1    4750 3500
-	1    0    0    -1
-$EndComp
-$Comp
-L CONN_1 TP13
-U 1 1 54105111
-P 3650 3650
-F 0 "TP13" H 3730 3650 40  0000 L CNN
-F 1 "CONN_1" H 3650 3705 30  0001 C CNN
-F 2 "" H 3650 3650 60  0000 C CNN
-F 3 "" H 3650 3650 60  0000 C CNN
-	1    3650 3650
-	1    0    0    -1
-$EndComp
-$Comp
-L CONN_1 TP12
-U 1 1 54105117
-P 3650 2100
-F 0 "TP12" H 3730 2100 40  0000 L CNN
-F 1 "CONN_1" H 3650 2155 30  0001 C CNN
-F 2 "" H 3650 2100 60  0000 C CNN
-F 3 "" H 3650 2100 60  0000 C CNN
-	1    3650 2100
-	1    0    0    -1
-$EndComp
 Wire Wire Line
 	3350 2650 3600 2650
@@
 	5650 2250 5650 2350
 Connection ~ 5650 2350
-Wire Wire Line
-	3600 1300 3600 1700
-Connection ~ 3600 1700
-Wire Wire Line
-	4500 2100 4500 2350
-Connection ~ 4500 2350
-Wire Wire Line
-	4600 3500 4600 3850
-Connection ~ 4600 3850
-Wire Wire Line
-	3500 2100 3500 2650
-Connection ~ 3500 2650
-Wire Wire Line
-	3500 3650 3500 4150
-Connection ~ 3500 4150
 $EndSCHEMATC
