File: Kicad/_autosave-HealthyPH.kicad_pcb (KiCad board)
At the start: 2 copper layers, 68.6 x 53.4 mm, 62 parts, among them CON1 LB_BarrelJack, P1 CONN_8, P2 WallWartExtension, Q1 TIP122, Q2 TIP122, U1 MCP6241, U2 MCP3901, U3 MC78L05, X1 CRYSTAL

Commit message: Layout ready for final check prior to PCB fab
Changed lines of the file:
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@@
   (layers
     (15 F.Cu signal)
-    (0 B.Cu signal)
+    (0 B.Cu signal hide)
     (16 B.Adhes user hide)
     (17 F.Adhes user)
@@
     (at 172.65 110.95 270)
     (attr smd)
-    (fp_text reference C11 (at 1.21 -1.46 270) (layer F.SilkS)
-      (effects (font (size 0.50038 0.50038) (thickness 0.10922)))
-    )
-    (fp_text value 1u (at -0.67 -1.41 270) (layer F.SilkS)
+    (fp_text reference C11 (at 2.8166 0.6666 360) (layer F.SilkS)
+      (effects (font (size 0.50038 0.50038) (thickness 0.10922)))
+    )
+    (fp_text value 1u (at 2.7658 -1.0352 360) (layer F.SilkS)
       (effects (font (size 0.50038 0.50038) (thickness 0.10922)))
     )
@@
     (at 180.2892 93.1672)
     (attr smd)
-    (fp_text reference R3 (at 0.8 -1.4) (layer F.SilkS)
-      (effects (font (size 0.50038 0.50038) (thickness 0.10922)))
-    )
-    (fp_text value 10K (at -0.8 -1.4) (layer F.SilkS)
+    (fp_text reference R3 (at 0.3683 1.9431) (layer F.SilkS)
+      (effects (font (size 0.50038 0.50038) (thickness 0.10922)))
+    )
+    (fp_text value 10K (at -1.143 1.8923) (layer F.SilkS)
       (effects (font (size 0.50038 0.50038) (thickness 0.10922)))
     )
@@
     (at 183.007 95.9612 90)
     (attr smd)
-    (fp_text reference R15 (at 0 -0.3175 90) (layer F.SilkS)
-      (effects (font (size 0.50038 0.50038) (thickness 0.10922)))
-    )
-    (fp_text value 10K (at 0 0.381 90) (layer F.SilkS)
-      (effects (font (size 0.50038 0.50038) (thickness 0.10922)))
-    )
+    (fp_text reference R15 (at -2.8702 -0.7493 180) (layer F.SilkS)
+      (effects (font (size 0.50038 0.50038) (thickness 0.10922)))
+    )
+    (fp_text value 10K (at -2.8194 1.1303 180) (layer F.SilkS)
+      (effects (font (size 0.50038 0.50038) (thickness 0.10922)))
+    )

Commit message: layout sent to OshPark
Parts:
- moved R13 44.6 mm to (210.3, 111.4), turned to 0 degrees
- moved R14 44.2 mm to (215.8, 111.6), turned to 0 degrees
- moved R12 42.9 mm to (205.6, 111.5), turned to 0 degrees
- moved D4 36.9 mm to (205.1, 108.0)
- moved TP12 14.9 mm to (202.5, 104.9)
- moved TP8 6.87 mm to (207.9, 90.2)
- moved R9 6.43 mm to (188.5, 73.0)
- moved TP15 5.45 mm to (210.1, 96.8)
- moved D5 4.86 mm to (206.4, 103.9)
- moved TP16 4.67 mm to (210.6, 105.8)
- moved D1 4.53 mm to (205.4, 95.9)
- moved R1 3.62 mm to (188.2, 101.5)
- moved R4 2.12 mm to (194.4, 90.0)
- moved TP11 1.58 mm to (202.1, 88.1)
- moved C1 1.50 mm to (193.2, 93.1)
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Connections:
- ARD1 pad 17: N-0000040 -> (no net)
- ARD1 pad 19: /Arduino/~CS -> (no net)
- ARD1 pad 20: N-0000044 -> (no net)
- ARD1 pad 21: N-0000042 -> /Arduino/~CS
- ARD1 pad 7: (no net) -> N-0000048
- ARD1 pad 8: (no net) -> N-0000045
- ARD1 pad 9: (no net) -> N-0000046
- D4 pad 1: N-0000036 -> N-0000038
- D4 pad 2: N-0000043 -> N-0000037
- D4 pad 3: N-0000045 -> N-0000036
- R12 pad 1: N-0000042 -> N-0000038
- R12 pad 2: N-0000036 -> N-0000048
- R13 pad 1: N-0000044 -> N-0000036
- R13 pad 2: N-0000043 -> N-0000045
- R14 pad 1: N-0000040 -> N-0000037
- R14 pad 2: N-0000045 -> N-0000046
Routing:
- net /Arduino/V+_ARD: track 130.6 -> 81.2 mm, vias 4 -> 3
- net N-0000026: track 9.15 -> 22.0 mm
- net N-0000037: track 0.00 -> 10.5 mm
- net N-0000045: track 13.6 -> 5.04 mm
- net N-0000046: track 0.00 -> 7.78 mm
- net N-0000042: track 4.68 -> 0.00 mm
- net N-0000040: track 4.38 -> 0.00 mm
- net N-0000048: track 0.00 -> 4.29 mm
- net /Pumps/SW_DownPump: track 19.0 -> 23.2 mm
- net N-0000038: track 0.00 -> 3.98 mm
- net /Digital Access/~CS_ISO: track 37.3 -> 33.3 mm, vias 2 -> 1
- net N-0000044: track 3.24 -> 0.00 mm
- net N-0000043: track 2.60 -> 0.00 mm
- net /Temperature/10K Therm: track 42.9 -> 45.5 mm
- net /Pumps/SW_UpPump: track 20.7 -> 23.3 mm
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