File: Kicad/_autosave-HealthyPH.kicad_pcb (KiCad board)
At the start: 2 copper layers, 68.6 x 53.4 mm, 48 parts, among them CON1 LB_BarrelJack, P1 CONN_8, P2 WallWartExtension, Q1 TIP122, Q2 TIP122, U1 MCP6241, U2 MCP3901, U3 MC78L05, X1 CRYSTAL

Commit message: Layout sent to OshPark
Parts:
- ~: renamed from ARD1; value ARDUINOPINS -> ~
- moved C10 10.9 mm to (197.9, 79.5), turned to 90 degrees
- moved D1 5.99 mm to (209.4, 100.3)
- moved C9 4.29 mm to (194.8, 83.7)
- moved D5 2.15 mm to (204.4, 104.7), turned to 0 degrees
- moved TP1 1.70 mm to (202.5, 84.9)
Routing:
- net /Arduino/V+_ARD: track 87.5 -> 98.4 mm, vias 1 -> 0
- net /Digital Access/V+_WallWart: track 145.6 -> 152.0 mm
- net AGND: track 59.2 -> 61.4 mm
- net /Pumps/SW_DownPump: track 23.2 -> 21.1 mm
- net /Pumps/SW_UpPump: track 23.3 -> 25.1 mm
- net /Digital Access/pH_ADC+: track 24.9 -> 23.1 mm

Commit message: before changing ADC
Parts:
- D1: value 4004 -> (none)
- moved D1 4.54 mm to (205.2, 98.7)
- moved D5 2.65 mm to (206.9, 104.0)
Routing:
- net /Arduino/V+_ARD: track 98.4 -> 93.6 mm
- net /Pumps/SW_DownPump: track 21.1 -> 20.1 mm
Changed lines of the file:
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@@
     (thickness 1.6)
     (drawings 11)
-    (tracks 381)
+    (tracks 377)
     (zones 0)
     (modules 48)
@@
   )
   (setup
-    (last_trace_width 0.6096)
+    (last_trace_width 0.254)
     (user_trace_width 0.254)
     (user_trace_width 0.6096)
@@
     (mod_text_size 1 1)
     (mod_text_width 0.15)
-    (pad_size 2.032 2.032)
-    (pad_drill 1.27)
+    (pad_size 1.524 2.54)
+    (pad_drill 1.016)
     (pad_to_mask_clearance 0)
     (aux_axis_origin 0 0)
@@
       (drillshape 0)
       (scaleselection 1)
-      (outputdirectory "//psf/Home/Documents/Lettuce Buddy HW/HealthyPH/Kicad/Gerbers/Dev Rev3/"))
+      (outputdirectory "//psf/Home/Documents/Lettuce Buddy HW/HealthyPH/Kicad/Gerbers/Dev Rev 2/"))
   )
   (net 0 "")
@@
   )
   (module "DO-214AC(SMA)" (layer F.Cu)
-    (at 209.423 100.2792 90)
+    (at 205.15072 98.73742 90)
     (descr "DO-214AC (SMA)  PACKAGE.")
     (tags "DO-214AC SMA")
     (attr smd)
-    (fp_text reference D1 (at 1 5 90) (layer F.SilkS)
+    (fp_text reference D1 (at -0.29718 3.20548 180) (layer F.SilkS)
       (effects (font (size 1.00076 1.00076) (thickness 0.11938)))
     )
-    (fp_text value 4004 (at 0.8 3.2 90) (layer F.SilkS)
+    (fp_text value "" (at 0.8 3.2 90) (layer F.SilkS)
       (effects (font (size 1.00076 1.00076) (thickness 0.11938)))
     )
@@
   )
   (module "DO-214AC(SMA)" (layer F.Cu)
-    (at 204.3938 104.7242)
+    (at 206.94142 104.013)
     (descr "DO-214AC (SMA)  PACKAGE.")
     (tags "DO-214AC SMA")
     (attr smd)
-    (fp_text reference D5 (at 0.8 4.4) (layer F.SilkS)
+    (fp_text reference D5 (at 3.64998 -2.0066) (layer F.SilkS)
       (effects (font (size 1.00076 1.00076) (thickness 0.11938)))
     )
@@
   (gr_line (start 217.04046 66.38544) (end 217.04046 77.81036) (angle 90) (layer Edge.Cuts) (width 0.1524))
   (gr_line (start 215.51646 64.86144) (end 217.04046 66.38544) (angle 90) (layer Edge.Cuts) (width 0.1524))
+  (segment (start 205.359 97.78492) (end 205.23708 97.78492) (width 0.254) (layer F.Cu) (net 0))
   (segment (start 172.07484 76.3016) (end 172.3136 76.3016) (width 0.254) (layer F.Cu) (net 1))
   (via (at 178.7906 69.8246) (size 0.6858) (layers F.Cu B.Cu) (net 1))
@@
   (segment (start 180.0606 71.1962) (end 180.0606 67.39636) (width 0.254) (layer F.Cu) (net 4))
   (segment (start 174.97298 76.28382) (end 180.0606 71.1962) (width 0.254) (layer F.Cu) (net 4))
-  (segment (start 206.29372 104.7242) (end 214.41344 104.7242) (width 0.6096) (layer F.Cu) (net 5))
-  (segment (start 214.41344 104.7242) (end 215.28798 103.84966) (width 0.6096) (layer F.Cu) (net 5))
-  (segment (start 209.423 98.37928) (end 209.423 97.2566) (width 0.6096) (layer F.Cu) (net 5))
-  (segment (start 209.423 97.2566) (end 209.8421 96.8375) (width 0.6096) (layer F.Cu) (net 5))
   (segment (start 196.90588 96.266) (end 214.503 96.266) (width 0.6096) (layer B.Cu) (net 5))
   (segment (start 215.38798 97.15098) (end 215.38798 97.36966) (width 0.6096) (layer B.Cu) (net 5))
   (segment (start 214.503 96.266) (end 215.38798 97.15098) (width 0.6096) (layer B.Cu) (net 5))
-  (segment (start 205.15072 96.8375) (end 209.8421 96.8375) (width 0.6096) (layer F.Cu) (net 5))
-  (segment (start 209.8421 96.8375) (end 214.85582 96.8375) (width 0.6096) (layer F.Cu) (net 5))
+  (segment (start 205.15072 96.8375) (end 214.85582 96.8375) (width 0.6096) (layer F.Cu) (net 5))
   (segment (start 214.85582 96.8375) (end 215.38798 97.36966) (width 0.6096) (layer F.Cu) (net 5))
+  (segment (start 208.84134 104.013) (end 215.12464 104.013) (width 0.6096) (layer F.Cu) (net 5))
   (segment (start 215.12464 104.013) (end 215.28798 103.84966) (width 0.6096) (layer F.Cu) (net 5))
   (segment (start 186.2709 97.5741) (end 187.6044 96.2406) (width 0.6096) (layer B.Cu) (net 5))
@@
   (segment (start 201.81 113.41) (end 201.801135 113.046535) (width 0.254) (layer F.Cu) (net 18))
   (segment (start 201.801135 113.046535) (end 201.8 113) (width 0.254) (layer F.Cu) (net 18))
-  (segment (start 209.423 102.17912) (end 198.92912 102.17912) (width 0.6096) (layer F.Cu) (net 19))
-  (segment (start 198.92912 102.17912) (end 197.55 100.8) (width 0.6096) (layer F.Cu) (net 19))
-  (segment (start 209.423 102.17912) (end 214.07852 102.17912) (width 0.6096) (layer F.Cu) (net 19))
-  (segment (start 214.07852 102.17912) (end 215.38798 100.86966) (width 0.6096) (layer F.Cu) (net 19))
+  (segment (start 205.15072 100.63734) (end 215.15566 100.63734) (width 0.6096) (layer F.Cu) (net 19))
+  (segment (start 215.15566 100.63734) (end 215.38798 100.86966) (width 0.6096) (layer F.Cu) (net 19))
+  (segment (start 197.55 100.8) (end 204.98806 100.8) (width 0.6096) (layer F.Cu) (net 19))
+  (segment (start 204.98806 100.8) (end 205.15072 100.63734) (width 0.6096) (layer F.Cu) (net 19))
   (segment (start 199.04992 102.29992) (end 197.55 100.8) (width 0.254) (layer F.Cu) (net 19))
-  (segment (start 202.49388 104.7242) (end 202.49388 106.25328) (width 0.6096) (layer F.Cu) (net 20))
-  (segment (start 214.64372 106.7054) (end 215.28798 107.34966) (width 0.6096) (layer F.Cu) (net 20))
-  (segment (start 202.946 106.7054) (end 214.64372 106.7054) (width 0.6096) (layer F.Cu) (net 20))
-  (segment (start 202.49388 106.25328) (end 202.946 106.7054) (width 0.6096) (layer F.Cu) (net 20))
-  (segment (start 197.55 108.6) (end 198.61808 108.6) (width 0.6096) (layer F.Cu) (net 20))
-  (segment (start 198.61808 108.6) (end 202.49388 104.7242) (width 0.6096) (layer F.Cu) (net 20))
+  (segment (start 215.28798 107.34966) (end 213.1051 107.34966) (width 0.6096) (layer F.Cu) (net 20))
+  (segment (start 207.3021 106.2736) (end 205.0415 104.013) (width 0.6096) (layer F.Cu) (net 20))
+  (segment (start 212.02904 106.2736) (end 207.3021 106.2736) (width 0.6096) (layer F.Cu) (net 20))
+  (segment (start 213.1051 107.34966) (end 212.02904 106.2736) (width 0.6096) (layer F.Cu) (net 20))
+  (segment (start 205.0415 104.013) (end 205.0415 104.49814) (width 0.6096) (layer F.Cu) (net 20))
+  (segment (start 200.93964 108.6) (end 197.55 108.6) (width 0.6096) (layer F.Cu) (net 20))
+  (segment (start 205.0415 104.49814) (end 200.93964 108.6) (width 0.6096) (layer F.Cu) (net 20))
   (segment (start 199.44992 110.49992) (end 197.55 108.6) (width 0.254) (layer F.Cu) (net 20) (status 30))
   (segment (start 215.2194 107.3268) (end 215.0732 107.3268) (width 0.254) (layer F.Cu) (net 20))
@@
   (segment (start 187.35972 92.28582) (end 188.87948 92.28582) (width 0.254) (layer F.Cu) (net 30))
   (segment (start 188.87948 92.28582) (end 189.84976 91.31554) (width 0.254) (layer F.Cu) (net 30))
-  (segment (start 172.8216 106.40568) (end 171.6786 106.40568) (width 0.6096) (layer F.Cu) (net 31))
-  (segment (start 172.8216 106.40568) (end 172.84192 106.40568) (width 0.6096) (layer F.Cu) (net 31))
-  (segment (start 175.2981 103.9495) (end 177.419 103.9495) (width 0.6096) (layer F.Cu) (net 31))
-  (segment (start 172.84192 106.40568) (end 175.2981 103.9495) (width 0.6096) (layer F.Cu) (net 31))
-  (segment (start 169.61866 102.54488) (end 169.61866 104.34574) (width 0.6096) (layer F.Cu) (net 31))
-  (segment (start 169.61866 104.34574) (end 171.6786 106.40568) (width 0.6096) (layer F.Cu) (net 31))
+  (segment (start 171.6786 106.40568) (end 174.96282 106.40568) (width 0.254) (layer F.Cu) (net 31))
+  (segment (start 174.96282 106.40568) (end 177.419 103.9495) (width 0.254) (layer F.Cu) (net 31))
+  (segment (start 169.61866 102.54488) (end 169.61866 104.34574) (width 0.254) (layer F.Cu) (net 31))
+  (segment (start 169.61866 104.34574) (end 171.6786 106.40568) (width 0.254) (layer F.Cu) (net 31))
   (segment (start 177.09642 104.27208) (end 177.419 103.9495) (width 0.254) (layer F.Cu) (net 31))
-  (segment (start 160.32734 110.63478) (end 165.80358 110.63478) (width 0.6096) (layer F.Cu) (net 32))
-  (segment (start 165.80358 110.63478) (end 168.529 113.3602) (width 0.6096) (layer F.Cu) (net 32))
+  (segment (start 160.32734 110.63478) (end 165.80358 110.63478) (width 0.254) (layer F.Cu) (net 32))
+  (segment (start 165.80358 110.63478) (end 168.529 113.3602) (width 0.254) (layer F.Cu) (net 32))
   (segment (start 168.529 113.3602) (end 168.529 113.35512) (width 0.254) (layer F.Cu) (net 32))
-  (segment (start 168.529 113.35512) (end 171.6786 110.20552) (width 0.6096) (layer F.Cu) (net 32))
+  (segment (start 168.529 113.35512) (end 171.6786 110.20552) (width 0.254) (layer F.Cu) (net 32))
   (segment (start 159.34182 94.12478) (end 162.47872 94.12478) (width 0.254) (layer F.Cu) (net 33))
   (segment (start 162.47872 94.12478) (end 162.90798 94.55404) (width 0.254) (layer F.Cu) (net 33))
